Commit message: Fix URDF mesh path to relative; update pybullet env path handling

File: robot_model/robot.urdf (robot description, URDF)
Before this commit: robot magnetic_robot, 1 links, 0 joints
Links:
- link base_link: geometry collision cylinder length=0.002 radius=0.0015; visual mesh filename=microrobot_ass.stl scale=1 1 1
